Commit message: 🦄 refactor(urdf, config, sim_env):

File: furniture_bench/assets/franka_description_ros/franka_description/robots/franka_panda.urdf (robot description, URDF)
Before this commit: robot panda, 20 links, 19 joints
Links:
- removed link panda_leftfinger
- removed link panda_link0_sc
- removed link panda_link1_sc
- removed link panda_link2_sc
- removed link panda_link3_sc
- removed link panda_link4_sc
- removed link panda_link5_sc
- removed link panda_link6_sc
- removed link panda_link7
- removed link panda_link7_sc
- removed link panda_rightfinger
- added link Left_Gripper, mass 0.11401; collision mesh filename=package://franka_description/robots/Gripper/meshes/Left_Gri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; visual mesh filename=package://franka_description/robots/Gripper/meshes/Left_Gri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
- added link Right_Gripper, mass 0.11017; collision mesh filename=package://franka_description/robots/Gripper/meshes/Right_Gr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; visual mesh filename=package://franka_description/robots/Gripper/meshes/Right_Gr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
- added link world
- link panda_hand: mass None -> 0.410076712822003; geometry collision mesh filename=package://franka_description/robots/Gripper/meshes/panda_ha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; visual mesh filename=package://franka_description/robots/Gripper/meshes/panda_ha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
- link panda_link0: mass 0.629769 -> 1.6185; geometry collision mesh filename=package://franka_description/robots/fr5v6/collision/base_li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; visual mesh filename=package://franka_description/robots/fr5v6/visual/base_link.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
- link panda_link1: mass 4.970684 -> 4.3771; geometry collision mesh filename=package://franka_description/robots/fr5v6/collision/j1_Link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; visual mesh filename=package://franka_description/robots/fr5v6/visual/j1_Link.DAE
- link panda_link2: mass 0.646926 -> 14.458; geometry collision mesh filename=package://franka_description/robots/fr5v6/collision/j2_Link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; visual mesh filename=package://franka_description/robots/fr5v6/visual/j2_Link.DAE
- link panda_link3: mass 3.228604 -> 7.6737; geometry collision mesh filename=package://franka_description/robots/fr5v6/collision/j3_Link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; visual mesh filename=package://franka_description/robots/fr5v6/visual/j3_Link.DAE
- link panda_link4: mass 3.587895 -> 1.6266; geometry collision mesh filename=package://franka_description/robots/fr5v6/collision/j4_Link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; visual mesh filename=package://franka_description/robots/fr5v6/visual/j4_Link.DAE
- link panda_link5: mass 1.225946 -> 1.5812; geometry collision mesh filename=package://franka_description/robots/fr5v6/collision/j5_Link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; visual mesh filename=package://franka_description/robots/fr5v6/visual/j5_Link.DAE
- link panda_link6: mass 1.666555 -> 0.52542; geometry collision mesh filename=package://franka_description/robots/fr5v6/collision/j6_Link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; visual mesh filename=package://franka_description/robots/fr5v6/visual/j6_Link.DAE
Joints:
- removed joint panda_finger_joint1
- removed joint panda_finger_joint2
- removed joint panda_joint3
- removed joint panda_joint4
- removed joint panda_joint5
- removed joint panda_joint6
- removed joint panda_joint7
- removed joint panda_link0_sc_joint
- removed joint panda_link1_sc_joint
- removed joint panda_link2_sc_joint
- removed joint panda_link3_sc_joint
- removed joint panda_link4_sc_joint
- removed joint panda_link5_sc_joint
- removed joint panda_link6_sc_joint
- removed joint panda_link7_sc_joint
- added joint LG: type prismatic, parent panda_hand, child Left_Gripper, origin xyz=0.071084 -0.02241 0.0801 rpy=0 0 0, axis 1 0 0, limit lower=0 upper=0.055 effort=10 velocity=0.1
- added joint RG: type prismatic, parent panda_hand, child Right_Gripper, origin xyz=-0.071084 0.01159 0.0801 rpy=0 0 -3.1416, axis 1 0 0, limit lower=0 upper=0.055 effort=10 velocity=0.1
- added joint panda_join3: type revolute, parent panda_link2, child panda_link3, origin xyz=-0.425 0 0 rpy=0 0 0, axis 0 0 1, limit lower=-2.8274 upper=2.8274 effort=150 velocity=3.15
- added joint panda_join4: type revolute, parent panda_link3, child panda_link4, origin xyz=-0.39501 0 0 rpy=0 0 0, axis 0 0 1, limit lower=-4.6251 upper=1.4835 effort=28 velocity=3.2
- added joint panda_join5: type revolute, parent panda_link4, child panda_link5, origin xyz=0 0 0.1021 rpy=1.5708 0 0, axis 0 0 1, limit lower=-3.0543 upper=3.0543 effort=28 velocity=3.2
- added joint panda_join6: type revolute, parent panda_link5, child panda_link6, origin xyz=0 0 0.102 rpy=-1.5708 0 0, axis 0 0 1, limit lower=-3.0543 upper=3.0543 effort=28 velocity=3.2
- added joint world: type fixed, parent world, child panda_link0
- joint panda_hand_joint: parent panda_link7 -> panda_link6
- joint panda_joint1: limit lower=-2.8973 upper=2.8973 effort=87.0 velocity=2.175 -> lower=-3.0543 upper=3.0543 effort=150 velocity=3.15; origin xyz=0 0 0.333 rpy=0 0 0 -> xyz=0 0 0 rpy=0 0 0
- joint panda_joint2: limit lower=-1.7628 upper=1.7628 effort=87.0 velocity=2.175 -> lower=-4.6251 upper=1.4835 effort=150 velocity=3.15; origin xyz=0 0 0 rpy=-1.5707963267948966 0 0 -> xyz=0 0 0.152 rpy=1.5708 0 0

File: furniture_bench/assets_no_tags/franka_description_ros/franka_description/robots/franka_panda.urdf (robot description, URDF)
Before this commit: robot panda, 20 links, 19 joints
Links:
- removed link panda_leftfinger
- removed link panda_link0_sc
- removed link panda_link1_sc
- removed link panda_link2_sc
- removed link panda_link3_sc
- removed link panda_link4_sc
- removed link panda_link5_sc
- removed link panda_link6_sc
- removed link panda_rightfinger
- added link Left_Gripper, mass 0.11401; collision mesh filename=package://franka_description/robots/Gripper/meshes/Left_Gri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; visual mesh filename=package://franka_description/robots/Gripper/meshes/Left_Gri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
- added link Right_Gripper, mass 0.11017; collision mesh filename=package://franka_description/robots/Gripper/meshes/Right_Gr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; visual mesh filename=package://franka_description/robots/Gripper/meshes/Right_Gr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
- added link world
- link panda_hand: mass None -> 0.410076712822003; geometry collision mesh filename=package://franka_description/robots/Gripper/meshes/panda_ha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; visual mesh filename=package://franka_description/robots/Gripper/meshes/panda_ha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
- link panda_link0: mass 0.629769 -> 1.6185; geometry collision mesh filename=package://franka_description/robots/fr5v6/collision/base_li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; visual mesh filename=package://franka_description/robots/fr5v6/visual/base_link.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
- link panda_link1: mass 4.970684 -> 4.3771; geometry collision mesh filename=package://franka_description/robots/fr5v6/collision/j1_Link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; visual mesh filename=package://franka_description/robots/fr5v6/visual/j1_Link.DAE
- link panda_link2: mass 0.646926 -> 14.458; geometry collision mesh filename=package://franka_description/robots/fr5v6/collision/j2_Link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; visual mesh filename=package://franka_description/robots/fr5v6/visual/j2_Link.DAE
- link panda_link3: mass 3.228604 -> 7.6737; geometry collision mesh filename=package://franka_description/robots/fr5v6/collision/j3_Link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; visual mesh filename=package://franka_description/robots/fr5v6/visual/j3_Link.DAE
- link panda_link4: mass 3.587895 -> 1.6266; geometry collision mesh filename=package://franka_description/robots/fr5v6/collision/j4_Link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; visual mesh filename=package://franka_description/robots/fr5v6/visual/j4_Link.DAE
- link panda_link5: mass 1.225946 -> 1.5812; geometry collision mesh filename=package://franka_description/robots/fr5v6/collision/j5_Link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; visual mesh filename=package://franka_description/robots/fr5v6/visual/j5_Link.DAE
- link panda_link6: mass 1.666555 -> 0.52542; geometry collision mesh filename=package://franka_description/robots/fr5v6/collision/j6_Link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; visual mesh filename=package://franka_description/robots/fr5v6/visual/j6_Link.DAE
Joints:
- removed joint panda_finger_joint1
- removed joint panda_finger_joint2
- removed joint panda_joint3
- removed joint panda_joint4
- removed joint panda_joint5
- removed joint panda_joint6
- removed joint panda_link0_sc_joint
- removed joint panda_link1_sc_joint
- removed joint panda_link2_sc_joint
- removed joint panda_link3_sc_joint
- removed joint panda_link4_sc_joint
- removed joint panda_link5_sc_joint
- removed joint panda_link6_sc_joint
- added joint LG: type prismatic, parent panda_hand, child Left_Gripper, origin xyz=0.071084 -0.02241 0.0801 rpy=0 0 0, axis 1 0 0, limit lower=0 upper=0.055 effort=10 velocity=0.1
- added joint RG: type prismatic, parent panda_hand, child Right_Gripper, origin xyz=-0.071084 0.01159 0.0801 rpy=0 0 -3.1416, axis 1 0 0, limit lower=0 upper=0.055 effort=10 velocity=0.1
- added joint panda_join3: type revolute, parent panda_link2, child panda_link3, origin xyz=-0.425 0 0 rpy=0 0 0, axis 0 0 1, limit lower=-2.8274 upper=2.8274 effort=150 velocity=3.15
- added joint panda_join4: type revolute, parent panda_link3, child panda_link4, origin xyz=-0.39501 0 0 rpy=0 0 0, axis 0 0 1, limit lower=-4.6251 upper=1.4835 effort=28 velocity=3.2
- added joint panda_join5: type revolute, parent panda_link4, child panda_link5, origin xyz=0 0 0.1021 rpy=1.5708 0 0, axis 0 0 1, limit lower=-3.0543 upper=3.0543 effort=28 velocity=3.2
- added joint panda_join6: type revolute, parent panda_link5, child panda_link6, origin xyz=0 0 0.102 rpy=-1.5708 0 0, axis 0 0 1, limit lower=-3.0543 upper=3.0543 effort=28 velocity=3.2
- added joint world: type fixed, parent world, child panda_link0
- joint panda_joint1: limit lower=-2.8973 upper=2.8973 effort=87.0 velocity=2.175 -> lower=-3.0543 upper=3.0543 effort=150 velocity=3.15; origin xyz=0 0 0.333 rpy=0 0 0 -> xyz=0 0 0 rpy=0 0 0
- joint panda_joint2: limit lower=-1.7628 upper=1.7628 effort=87.0 velocity=2.175 -> lower=-4.6251 upper=1.4835 effort=150 velocity=3.15; origin xyz=0 0 0 rpy=-1.5707963267948966 0 0 -> xyz=0 0 0.152 rpy=1.5708 0 0

Commit message: 🦄 refactor(urdf):
changed urdf for realman gen72

File: furniture_bench/assets/franka_description_ros/franka_description/robots/franka_panda.urdf (robot description, URDF)
Before this commit: robot panda, 20 links, 19 joints
Links:
- removed link panda_link0_sc
- removed link panda_link1_sc
- removed link panda_link2_sc
- removed link panda_link3_sc
- removed link panda_link4_sc
- removed link panda_link5_sc
- removed link panda_link6_sc
- removed link panda_link7_sc
- link panda_hand: mass None -> 0.410076712822003; geometry collision mesh filename=package://franka_description/robots/Gripper/meshes/panda_ha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; visual mesh filename=package://franka_description/robots/Gripper/meshes/panda_ha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
- link panda_leftfinger: mass None -> 0.11401; geometry collision box size=4e-2 3.5e-2 13.5e-2; visual mesh filename=package://franka_description/robots/Gripper/meshes/Left_Gri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
- link panda_link0: mass 0.629769 -> 0.725732279372378; geometry collision mesh filename=package://franka_description/robots/meshes_gen/base_link.STL; visual mesh filename=package://franka_description/robots/meshes_gen/base_link.dae
- link panda_link1: mass 4.970684 -> 0.511231576042974; geometry collision mesh filename=package://franka_description/robots/meshes_gen/Link1.STL; visual mesh filename=package://franka_description/robots/meshes_gen/Link1.dae
- link panda_link2: mass 0.646926 -> 0.551907023014854; geometry collision mesh filename=package://franka_description/robots/meshes_gen/Link2.STL; visual mesh filename=package://franka_description/robots/meshes_gen/Link2.dae
- link panda_link3: mass 3.228604 -> 0.774130450031718; geometry collision mesh filename=package://franka_description/robots/meshes_gen/Link3.STL; visual mesh filename=package://franka_description/robots/meshes_gen/Link3.dae
- link panda_link4: mass 3.587895 -> 0.437130215853825; geometry collision mesh filename=package://franka_description/robots/meshes_gen/Link4.STL; visual mesh filename=package://franka_description/robots/meshes_gen/Link4.dae
- link panda_link5: mass 1.225946 -> 0.424276753764529; geometry collision mesh filename=package://franka_description/robots/meshes_gen/Link5.STL; visual mesh filename=package://franka_description/robots/meshes_gen/Link5.dae
- link panda_link6: mass 1.666555 -> 0.302793039332829; geometry collision mesh filename=package://franka_description/robots/meshes_gen/Link6.STL; visual mesh filename=package://franka_description/robots/meshes_gen/Link6.dae
- link panda_link7: mass 0.735522 -> 0.176612671882913; geometry collision mesh filename=package://franka_description/robots/meshes_gen/Link7.STL; visual mesh filename=package://franka_description/robots/meshes_gen/Link7.dae
- link panda_rightfinger: mass None -> 0.11017; geometry collision box size=4e-2 3.5e-2 13.5e-2; visual mesh filename=package://franka_description/robots/Gripper/meshes/Right_Gr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
Joints:
- removed joint panda_finger_joint1
- removed joint panda_finger_joint2
- removed joint panda_joint7
- removed joint panda_link0_sc_joint
- removed joint panda_link1_sc_joint
- removed joint panda_link2_sc_joint
- removed joint panda_link3_sc_joint
- removed joint panda_link4_sc_joint
- removed joint panda_link5_sc_joint
- removed joint panda_link6_sc_joint
- removed joint panda_link7_sc_joint
- added joint LG: type prismatic, parent panda_hand, child panda_leftfinger, origin xyz=0.125 -0.02241 0.0801 rpy=0 0 0, axis -1 0 0, limit lower=0 upper=0.055 effort=10 velocity=0.1
- added joint RG: type prismatic, parent panda_hand, child panda_rightfinger, origin xyz=-0.125 0.01159 0.0801 rpy=0 0 -3.1416, axis -1 0 0, limit lower=0 upper=0.055 effort=10 velocity=0.1
- added joint panda_join7: type revolute, parent panda_link6, child panda_link7, origin xyz=0.0905 0.067 0 rpy=1.5708 0 1.5708, axis 0 0 1, limit lower=-3.0014 upper=3.0014 effort=5 velocity=3.926
- joint panda_hand_joint: origin xyz=0 0 0.107 rpy=0 0 -0.785398163397 -> xyz=0 0 0 rpy=0 0 0
- joint panda_joint1: limit lower=-2.8973 upper=2.8973 effort=87.0 velocity=2.175 -> lower=-3.0014 upper=3.0014 effort=25 velocity=3.141; origin xyz=0 0 0.333 rpy=0 0 0 -> xyz=0 0 0.218 rpy=0 0 0
- joint panda_joint2: limit lower=-1.7628 upper=1.7628 effort=87.0 velocity=2.175 -> lower=-1.8323 upper=1.8323 effort=25 velocity=3.141; origin xyz=0 0 0 rpy=-1.5707963267948966 0 0 -> xyz=0 0 0 rpy=-1.5708 0 0
- joint panda_joint3: limit lower=-2.8973 upper=2.8973 effort=87.0 velocity=2.175 -> lower=-3.0014 upper=3.0014 effort=25 velocity=3.141; origin xyz=0 -0.316 0 rpy=1.5707963267948966 0 0 -> xyz=0 -0.28 0 rpy=1.5708 0 0
- joint panda_joint4: limit lower=-3.0718 upper=-0.0698 effort=87.0 velocity=2.175 -> lower=-2.8792 upper=0.9597 effort=25 velocity=3.141; origin xyz=0.0825 0 0 rpy=1.5707963267948966 0 0 -> xyz=0.04 0 0 rpy=1.5708 0 0
- joint panda_joint5: limit lower=-2.8973 upper=2.8973 effort=12.0 velocity=2.61 -> lower=-3.0014 upper=3.0014 effort=5 velocity=3.926; origin xyz=-0.0825 0.384 0 rpy=-1.5707963267948966 0 0 -> xyz=-0.019 0.2525 0 rpy=-1.5708 0 0
- joint panda_joint6: limit lower=-0.0175 upper=3.7525 effort=12.0 velocity=2.61 -> lower=-1.707 upper=1.783 effort=5 velocity=3.926; origin xyz=0 0 0 rpy=1.5707963267948966 0 0 -> xyz=0 0 0 rpy=1.5708 0 0

File: furniture_bench/assets_no_tags/franka_description_ros/franka_description/robots/franka_panda.urdf (robot description, URDF)
Before this commit: robot panda, 20 links, 19 joints
Links:
- removed link panda_link0_sc
- removed link panda_link1_sc
- removed link panda_link2_sc
- removed link panda_link3_sc
- removed link panda_link4_sc
- removed link panda_link5_sc
- removed link panda_link6_sc
- removed link panda_link7_sc
- link panda_link0: mass 0.629769 -> 0.725732279372378; geometry collision mesh filename=package://franka_description/robots/meshes_gen/base_link.STL; visual mesh filename=package://franka_description/robots/meshes_gen/base_link.dae
- link panda_link1: mass 4.970684 -> 0.511231576042974; geometry collision mesh filename=package://franka_description/robots/meshes_gen/Link1.STL; visual mesh filename=package://franka_description/robots/meshes_gen/Link1.dae
- link panda_link2: mass 0.646926 -> 0.551907023014854; geometry collision mesh filename=package://franka_description/robots/meshes_gen/Link2.STL; visual mesh filename=package://franka_description/robots/meshes_gen/Link2.dae
- link panda_link3: mass 3.228604 -> 0.774130450031718; geometry collision mesh filename=package://franka_description/robots/meshes_gen/Link3.STL; visual mesh filename=package://franka_description/robots/meshes_gen/Link3.dae
- link panda_link4: mass 3.587895 -> 0.437130215853825; geometry collision mesh filename=package://franka_description/robots/meshes_gen/Link4.STL; visual mesh filename=package://franka_description/robots/meshes_gen/Link4.dae
- link panda_link5: mass 1.225946 -> 0.424276753764529; geometry collision mesh filename=package://franka_description/robots/meshes_gen/Link5.STL; visual mesh filename=package://franka_description/robots/meshes_gen/Link5.dae
- link panda_link6: mass 1.666555 -> 0.302793039332829; geometry collision mesh filename=package://franka_description/robots/meshes_gen/Link6.STL; visual mesh filename=package://franka_description/robots/meshes_gen/Link6.dae
- link panda_link7: mass 0.735522 -> 0.176612671882913; geometry collision mesh filename=package://franka_description/robots/meshes_gen/Link7.STL; visual mesh filename=package://franka_description/robots/meshes_gen/Link7.dae
Joints:
- removed joint panda_joint7
- removed joint panda_link0_sc_joint
- removed joint panda_link1_sc_joint
- removed joint panda_link2_sc_joint
- removed joint panda_link3_sc_joint
- removed joint panda_link4_sc_joint
- removed joint panda_link5_sc_joint
- removed joint panda_link6_sc_joint
- removed joint panda_link7_sc_joint
- added joint panda_join7: type revolute, parent panda_link6, child panda_link7, origin xyz=0.0905 0.067 0 rpy=1.5708 0 1.5708, axis 0 0 1, limit lower=-3.0014 upper=3.0014 effort=5 velocity=3.926
- joint panda_joint1: limit lower=-2.8973 upper=2.8973 effort=87.0 velocity=2.175 -> lower=-3.0014 upper=3.0014 effort=25 velocity=3.141; origin xyz=0 0 0.333 rpy=0 0 0 -> xyz=0 0 0.218 rpy=0 0 0
- joint panda_joint2: limit lower=-1.7628 upper=1.7628 effort=87.0 velocity=2.175 -> lower=-1.8323 upper=1.8323 effort=25 velocity=3.141; origin xyz=0 0 0 rpy=-1.5707963267948966 0 0 -> xyz=0 0 0 rpy=-1.5708 0 0
- joint panda_joint3: limit lower=-2.8973 upper=2.8973 effort=87.0 velocity=2.175 -> lower=-3.0014 upper=3.0014 effort=25 velocity=3.141; origin xyz=0 -0.316 0 rpy=1.5707963267948966 0 0 -> xyz=0 -0.28 0 rpy=1.5708 0 0
- joint panda_joint4: limit lower=-3.0718 upper=-0.0698 effort=87.0 velocity=2.175 -> lower=-2.8792 upper=0.9597 effort=25 velocity=3.141; origin xyz=0.0825 0 0 rpy=1.5707963267948966 0 0 -> xyz=0.04 0 0 rpy=1.5708 0 0
- joint panda_joint5: limit lower=-2.8973 upper=2.8973 effort=12.0 velocity=2.61 -> lower=-3.0014 upper=3.0014 effort=5 velocity=3.926; origin xyz=-0.0825 0.384 0 rpy=-1.5707963267948966 0 0 -> xyz=-0.019 0.2525 0 rpy=-1.5708 0 0
- joint panda_joint6: limit lower=-0.0175 upper=3.7525 effort=12.0 velocity=2.61 -> lower=-1.707 upper=1.783 effort=5 velocity=3.926; origin xyz=0 0 0 rpy=1.5707963267948966 0 0 -> xyz=0 0 0 rpy=1.5708 0 0

Commit message: changed 10.21

File: furniture_bench/assets/franka_description_ros/franka_description/robots/franka_panda.urdf (robot description, URDF)
Before this commit: robot panda, 9 links, 8 joints
Links:
- removed link panda_link7_sc
- added link panda_link4, mass 0.437130215853825; collision mesh filename=package://franka_description/robots/meshes_gen/Link4.STL; visual mesh filename=package://franka_description/robots/meshes_gen/Link4.dae
- added link panda_link5, mass 0.424276753764529; collision mesh filename=package://franka_description/robots/meshes_gen/Link5.STL; visual mesh filename=package://franka_description/robots/meshes_gen/Link5.dae
- added link panda_link6, mass 0.302793039332829; collision mesh filename=package://franka_description/robots/meshes_gen/Link6.STL; visual mesh filename=package://franka_description/robots/meshes_gen/Link6.dae
- added link panda_link7, mass 0.176612671882913; collision mesh filename=package://franka_description/robots/meshes_gen/Link7.STL; visual mesh filename=package://franka_description/robots/meshes_gen/Link7.dae
- link panda_hand: mass None -> 0.410076712822003
- link panda_leftfinger: mass None -> 0.11401; geometry collision box size=4e-2 3.5e-2 13.5e-2; visual mesh filename=package://franka_description/robots/Gripper/meshes/Left_Gri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
- link panda_link1: mass 0.629769 -> 0.511231576042974
- link panda_link3: mass 0.646926 -> 0.774130450031718; geometry collision mesh filename=package://franka_description/robots/meshes_gen/Link3.STL; visual mesh filename=package://franka_description/robots/meshes_gen/Link3.dae
- link panda_rightfinger: mass None -> 0.11017; geometry collision box size=4e-2 3.5e-2 13.5e-2; visual mesh filename=package://franka_description/robots/Gripper/meshes/Right_Gr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
Joints:
- removed joint panda_finger_joint1
- removed joint panda_finger_joint2
- removed joint panda_joint7
- removed joint panda_link7_sc_joint
- added joint LG: type prismatic, parent panda_hand, child panda_leftfinger, origin xyz=0.125 -0.02241 0.0801 rpy=0 0 0, axis -1 0 0, limit lower=0 upper=0.055 effort=10 velocity=0.1
- added joint RG: type prismatic, parent panda_hand, child panda_rightfinger, origin xyz=-0.125 0.01159 0.0801 rpy=0 0 -3.1416, axis -1 0 0, limit lower=0 upper=0.055 effort=10 velocity=0.1
- added joint panda_join7: type revolute, parent panda_link6, child panda_link7, origin xyz=0.0905 0.067 0 rpy=1.5708 0 1.5708, axis 0 0 1, limit lower=-3.0014 upper=3.0014 effort=5 velocity=3.926
- added joint panda_joint3: type revolute, parent panda_link2, child panda_link3, origin xyz=0 -0.28 0 rpy=1.5708 0 0, axis 0 0 1, limit lower=-3.0014 upper=3.0014 effort=25 velocity=3.141
- added joint panda_joint4: type revolute, parent panda_link3, child panda_link4, origin xyz=0.04 0 0 rpy=1.5708 0 0, axis 0 0 1, limit lower=-2.8792 upper=0.9597 effort=25 velocity=3.141
- added joint panda_joint5: type revolute, parent panda_link4, child panda_link5, origin xyz=-0.019 0.2525 0 rpy=-1.5708 0 0, axis 0 0 1, limit lower=-3.0014 upper=3.0014 effort=5 velocity=3.926
- added joint panda_joint6: type revolute, parent panda_link5, child panda_link6, origin xyz=0 0 0 rpy=1.5708 0 0, axis 0 0 1, limit lower=-1.707 upper=1.783 effort=5 velocity=3.926
- joint panda_hand_joint: parent panda_link6 -> panda_link7
