Commit message: ✨ feat(config,urdf): change para

File: furniture_bench/assets/franka_description_ros/franka_description/robots/franka_panda (changed).urdf (robot description, URDF)
Before this commit: robot panda, 12 links, 11 joints
Links:
- link panda_leftfinger: geometry collision box size=1.43e-2 2.58e-2 1.60e-2; collision box size=2.26e-2 2.58e-2 2.09e-2
- link panda_rightfinger: geometry collision box size=1.43e-2 2.58e-2 1.60e-2; collision box size=2.26e-2 2.58e-2 2.09e-2
Joints:
- joint panda_hand_joint: origin xyz=0 0 0 rpy=0 0 -0.785398163397 -> xyz=0 0 0 rpy=0 0 0

File: furniture_bench/assets/franka_description_ros/franka_description/robots/franka_panda.urdf (robot description, URDF)
Before this commit: robot panda, 12 links, 11 joints
Links:
- link panda_leftfinger: geometry collision box size=1.43e-2 2.58e-2 1.60e-2; collision box size=2.26e-2 2.58e-2 2.09e-2
- link panda_rightfinger: geometry collision box size=1.43e-2 2.58e-2 1.60e-2; collision box size=2.26e-2 2.58e-2 2.09e-2
